File: ORION_boost_v3.kicad_sch (KiCad schematic)
At the start: 141 parts, among them J1 Conn_02x04_Odd_Even, J2 Conn_01x10, J3 Conn_01x03, J4 Conn_01x03, J5 Conn_01x01, J6 Conn_01x01, J7 Conn_01x02, J8 Conn_01x02, J9 Conn_01x02, P1 CONN_01X06, P2 CONN_01X02, P3 CONN_01X02, P4 CONN_01X02, P5 CONN_01X02, P6 CONN_01X02, P7 CONN_01X02, Q1 Q_NMOS_GDS, Q2 Q_NMOS_GDS, Q3 Q_NMOS_GSD, Q4 Q_PMOS_GDS, Q5 Q_NMOS_GDS, Q6 Q_NMOS_GDS, Q7 Q_NMOS_GDS, Q8 Q_NMOS_GDS, Q9 Q_NMOS_GDS, SW1 SW_Push, SW2 SW_Push, SW3 SW_Push, U1 STM32F303CBTx, U2 LTC2875-S8, U4 INA199, X1 ceralock

Commit message: 天丼マン
Parts:
- removed D6: D, Diode_SMD:D_0603_1608Metric, symbol SSL_BST_ver1.3-rescue:D
- added D6: D, Diode_SMD:D_PowerDI-123, symbol Device:D
- added Q10: Q_NMOS_GSD, Package_TO_SOT_SMD:SOT-23, symbol Device:Q_NMOS_GSD
- added R41: 100, Resistor_SMD:R_0603_1608Metric, symbol Device:R
- added R42: 1k, Resistor_SMD:R_0603_1608Metric, symbol Device:R
Connections:
- net SW1 is gone; now on net SW_1: SW2.1
- net SW2 is gone; now on net SW_2: SW3.1
- net GND: now also Q10.2 (S), R42.1
- net LED_CURRENT: now also R41.2
- net TEMP_FET: now also C10.2, R11.1, TH1.2
- net at D10.1 (K), D14.1 (K): now also D6.2 (A)
- net TEMP_COIL_3: no longer names the net of U1.28 (PB15)
- new net: Q10.1 (G), R41.1, R42.2
- new net: D6.1 (K), Q10.3 (D)
- no-connect marks 4 -> 5
Other:
- moved on the sheet: D10, D11, D12, D13, D14, D7, D8, D9
