File: ORION_boost_v5.kicad_sch (KiCad schematic)
At the start: 154 parts, among them J1 Conn_02x04_Odd_Even, J10 Conn_01x01, J11 Conn_01x01, J2 Conn_01x10, J3 Conn_01x03, J4 Conn_01x03, J5 Conn_01x01, J6 Conn_01x01, J7 Conn_01x02, J8 Conn_01x02, J9 Conn_01x02, P1 CONN_01X06, P2 CONN_01X02, P3 CONN_01X02, P4 CONN_01X02, P5 CONN_01X02, P6 CONN_01X02, P7 CONN_01X02, Q1 Q_NMOS_GDS, Q10 Q_NMOS_GSD, Q2 Q_NMOS_GDS, Q3 Q_NMOS_GSD, Q4 Q_PMOS_GDS, Q5 Q_NMOS_GDS, Q6 Q_NMOS_GDS, Q7 Q_NMOS_GDS, Q8 Q_NMOS_GDS, Q9 Q_NMOS_GDS, SW1 SW_Push, SW2 SW_Push, SW3 SW_Push, SW4 SW_Push, U1 STM32F303CBTx, U2 MAX3051, U3 ZXCT108x, X1 ceralock

Commit message: KiCAD8.0に更新
Parts:
- removed FB1: FerriteBead, Resistor_SMD:R_0603_1608Metric, symbol Device:FerriteBead
- added F4: Fuse, Fuse:Fuse_1210_3225Metric, symbol Device:Fuse
- added R45: 1, Resistor_SMD:R_0603_1608Metric, symbol SSL_BST_ver1.3-rescue:R
- SW1, SW2, SW3, SW4: footprint Button_Switch_SMD:SW_Push_1P1T_NO_CK_KMR2 -> Button_Switch_SMD:SW_Push_SPST_NO_Alps_SKRK
Connections:
- net +3.3V: now also R45.2
- net +BATT: now also F4.2
- net at D18.2 (A), D27.1 (K), F3.1: now also F4.1
- net at C1.2, U1.9 (VDDA): now also R45.1
Other:
- moved on the sheet: D18, F3, R35

Commit message: KiCAD8に更新
Parts:
- added J12: Conn_01x02, Connector_JST:JST_PH_B2B-PH-K_1x02_P2.00mm_Vertical, symbol Connector_Generic:Conn_01x02
Connections:
- net GND: now also J12.1 (Pin_1)
- net LOGIC_POWER: now also J12.2 (Pin_2)
Changed lines of the file:
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@@
 		)
 	)
+	(label "LOGIC_POWER"
+		(at 300.99 320.04 180)
+		(fields_autoplaced yes)
+		(effects
+			(font
+				(size 1.27 1.27)
+			)
+			(justify right bottom)
+		)
+	)
 	(label "KICK_1_GATE"
 		(at 368.3 97.79 0)
@@
 			)
 		)
-		(property "Description" ""
+		(property "Description" "S3AB"
 			(at 401.32 303.53 0)
 			(effects
@@
 			)
 		)
-		(property "Description" ""
+		(property "Description" "S3AB"
 			(at 351.79 298.45 0)
 			(effects
@@
 			)
 		)
-		(property "Description" ""
+		(property "Description" "IPD60R180P7S"
 			(at 406.4 107.95 0)
 			(effects
@@
 			)
 		)
-		(property "Description" ""
+		(property "Description" "IPD60R180P7S"
 			(at 471.17 165.1 0)
 			(effects
@@
 	)
 	(symbol
+		(lib_id "Connector_Generic:Conn_01x02")
+		(at 306.07 317.5 0)
+		(unit 1)
+		(exclude_from_sim no)
+		(in_bom yes)
+		(on_board yes)
+		(dnp no)
+		(fields_autoplaced yes)
+		(property "Reference" "J12"
+			(at 308.61 317.4999 0)
+			(effects
+				(font
+					(size 1.27 1.27)
+				)
+				(justify left)
+			)
+		)
+		(property "Value" "Conn_01x02"
+			(at 308.61 320.0399 0)
+			(effects
+				(font
+					(size 1.27 1.27)
+				)
+				(justify left)
+			)
+		)
+		(property "Footprint" "Connector_JST:JST_PH_B2B-PH-K_1x02_P2.00mm_Vertical"
+			(at 306.07 317.5 0)
+			(effects
+				(font
+					(size 1.27 1.27)
+				)
+				(hide yes)
+			)
+		)
+		(property "Datasheet" "~"
+			(at 306.07 317.5 0)
+			(effects
+				(font
+					(size 1.27 1.27)
+				)
+				(hide yes)
+			)
+		)
+		(property "Description" "Generic connector, single row, 01x02, script generated (kicad-library-utils/schlib/autogen/connector/)"
+			(at 306.07 317.5 0)
+			(effects
+				(font
+					(size 1.27 1.27)
+				)
+				(hide yes)
+			)
+		)
+		(pin "2"
+		)
+		(pin "1"
+		)
+		(instances
+			(project ""
+				(path "/a24ddb4f-c217-42ca-b6cb-d12da84fb2b9"
+					(reference "J12")
+					(unit 1)
+				)
+			)
+		)
+	)
+	(symbol
 		(lib_id "power:+12V")
 		(at 358.14 229.87 0)
@@
 			)
 		)
-		(property "Description" ""
+		(property "Description" "UDZVTE-1712B"
 			(at 406.4 322.58 0)
 			(effects
@@
 			)
 		)
-		(property "Description" ""
+		(property "Description" "IPD60R180P7S"
 			(at 440.69 107.95 0)
 			(effects
@@
 	)
 	(symbol
+		(lib_id "SSL_BST_ver1.3_rev2-rescue:GND-power")
+		(at 300.99 317.5 270)
+		(unit 1)
+		(exclude_from_sim no)
+		(in_bom yes)
+		(on_board yes)
+		(dnp no)
+		(property "Reference" "#PWR039"
+			(at 294.64 317.5 0)
+			(effects
+				(font
+					(size 1.27 1.27)
+				)
+				(hide yes)
+			)
+		)
+		(property "Value" "GND"
+			(at 296.5958 317.627 0)
+			(effects
+				(font
+					(size 1.27 1.27)
+				)
+			)
+		)
+		(property "Footprint" ""
+			(at 300.99 317.5 0)
+			(effects
+				(font
+					(size 1.27 1.27)
+				)
+				(hide yes)
+			)
+		)
+		(property "Datasheet" ""
+			(at 300.99 317.5 0)
+			(effects
+				(font
+					(size 1.27 1.27)
+				)
+				(hide yes)
+			)
+		)
+		(property "Description" ""
+			(at 300.99 317.5 0)
+			(effects
+				(font
+					(size 1.27 1.27)
+				)
+				(hide yes)
+			)
+		)
+		(pin "1"
+		)
+		(instances
+			(project "ORION_boost_v5"
+				(path "/a24ddb4f-c217-42ca-b6cb-d12da84fb2b9"
+					(reference "#PWR039")
+					(unit 1)
+				)
+			)
+		)
+	)
+	(symbol
 		(lib_id "SSL_BST_ver1.3-rescue:C")
 		(at 355.6 292.1 90)
@@
 			)
 		)
-		(property "Description" ""
+		(property "Description" "IPD60R180P7S"
 			(at 402.59 165.1 0)
 			(effects
@@
 			)
 		)
-		(property "Description" ""
+		(property "Description" "BSS138"
 			(at 411.48 354.33 0)
 			(effects
@@
 			)
 		)
-		(property "Description" ""
+		(property "Description" "IPD60R180P7S"
 			(at 433.07 165.1 0)
 			(effects
@@
 			)
 		)
-		(property "Description" ""
+		(property "Description" "IPD60R180P7S"
 			(at 473.71 107.95 0)
 			(effects
